Commit message: first commit custom drone

File: rotors_description/urdf/component_snippets.xacro (robot description, xacro)
@@ -17,4 +17,5 @@
 -->
 <robot xmlns:xacro="http://ros.org/wiki/xacro">
+  <xacro:property name="pi" value="3.14159265359" />
   <!-- Macro to add logging to a bag file. -->
   <xacro:macro name="bag_plugin_macro"
@@ -562,5 +563,5 @@
       image_width="752"
       image_height="480"
-      image_format="L8"
+      image_format="R8G8B8"
       min_distance="0.02"
       max_distance="30"
@@ -583,5 +584,5 @@
       image_width="752"
       image_height="480"
-      image_format="L8"
+      image_format="R8G8B8"
       min_distance="0.02"
       max_distance="${max_range}"
@@ -630,7 +631,7 @@
         <update_rate>${frame_rate}</update_rate>
         <camera>
-          <horizontal_fov>2</horizontal_fov>
+          <horizontal_fov>1.2</horizontal_fov>
           <image>
-            <format>L8</format>
+            <format>R8G8B8</format>
             <width>640</width>
             <height>480</height>
@@ -664,4 +665,73 @@
     </gazebo>
   </xacro:macro>
+  <!-- Macro to add a depth camera on the Picoflexx. -->
+  <xacro:macro name="picoflexx_depth_macro"
+    params="namespace parent_link camera_suffix frame_rate max_range *origin">
+    <link name="${namespace}/camera_${camera_suffix}_link">
+      <collision>
+        <origin xyz="0 0 0" rpy="0 0 0" />
+        <geometry>
+          <cylinder length="0.01" radius="0.007" />
+        </geometry>
+      </collision>
+      <inertial>
+        <mass value="1e-5" />
+        <origin xyz="0 0 0" rpy="0 0 0" />
+        <inertia ixx="1e-6" ixy="0" ixz="0" iyy="1e-6" iyz="0" izz="1e-6" />
+      </inertial>
+    </link>
+    <joint name="${namespace}/camera_${camera_suffix}_joint" type="fixed">
+      <xacro:insert_block name="origin" />
+      <parent link="${parent_link}" />
+      <child link="${namespace}/camera_${camera_suffix}_link" />
+      <limit upper="0" lower="0" effort="0" velocity="0" />
+    </joint>
+    <!-- Optical center of camera -->
+    <link name="${namespace}/camera_${camera_suffix}_optical_center_link" />
+    <joint name="${namespace}/camera_${camera_suffix}_optical_center_joint" type="fixed">
+      <origin xyz="0 0 0" rpy="${-pi/2} 0 ${-pi/2}" />
+      <parent link="${namespace}/camera_${camera_suffix}_link" />
+      <child link="${namespace}/camera_${camera_suffix}_optical_center_link" />
+      <limit upper="0" lower="0" effort="0" velocity="0" />
+    </joint>
+    <gazebo reference="${namespace}/camera_${camera_suffix}_link">
+      <sensor type="depth" name="${namespace}_camera_{camera_suffix}">
+        <always_on>true</always_on>
+        <update_rate>${frame_rate}</update_rate>
+        <camera>
+          <horizontal_fov>1.2</horizontal_fov>
+          <image>
+            <format>R8G8B8</format>
+            <width>360</width>
+            <height>480</height>
+          </image>
+          <clip>
+            <near>0.01</near>
+            <far>${max_range}</far>
+          </clip>
+        </camera>
+        <plugin name="${namespace}_camera_{camera_suffix}" filename="libgazebo_ros_openni_kinect.so">
+          <robotNamespace>${namespace}</robotNamespace>
+          <alwaysOn>true</alwaysOn>
+          <baseline>0.11</baseline>
+          <updateRate>${frame_rate}</updateRate>
+          <cameraName>camera_${camera_suffix}</cameraName>
+          <imageTopicName>camera/image_raw</imageTopicName>
+          <cameraInfoTopicName>camera/camera_info</cameraInfoTopicName>
+          <depthImageTopicName>depth/disparity</depthImageTopicName>
+          <depthImageCameraInfoTopicName>depth/camera_info</depthImageCameraInfoTopicName>
+          <pointCloudTopicName>depth/points</pointCloudTopicName>
+          <frameName>camera_${camera_suffix}_optical_center_link</frameName>
+          <pointCloudCutoff>0.5</pointCloudCutoff>
+          <pointCloudCutoffMax>${max_range}</pointCloudCutoffMax>
+          <distortionK1>0.0</distortionK1>
+          <distortionK2>0.0</distortionK2>
+          <distortionK3>0.0</distortionK3>
+          <distortionT1>0.0</distortionT1>
+          <distortionT2>0.0</distortionT2>
+        </plugin>
+      </sensor>
+    </gazebo>
+  </xacro:macro>
   <!-- VI-Sensor Macro -->
   <xacro:macro name="vi_sensor_macro" params="namespace parent_link enable_cameras enable_depth enable_ground_truth *origin">
@@ -704,5 +774,5 @@
       <xacro:vi_sensor_depth_macro
         namespace="${namespace}" parent_link="${namespace}/vi_sensor_link"
-        camera_suffix="depth" frame_rate="30.0" max_range="10.0">
+        camera_suffix="depth" frame_rate="30.0" max_range="7.0">
         <origin xyz="0.015 0.055 0.0065" rpy="0 0 0" />
       </xacro:vi_sensor_depth_macro>
@@ -760,4 +830,72 @@
     </xacro:imu_plugin_macro>
   </xacro:macro>
+    <!-- Picoflexx Macro -->
+  <xacro:macro name="picoflexx_macro" params="namespace parent_link enable_cameras enable_depth enable_ground_truth *origin">
+    <!-- Picoflexx Sensor Link -->
+    <link name="${namespace}/picoflexx_link">
+      <collision>
+        <origin xyz="0 0 0" rpy="0 0 0" />
+        <geometry>
+          <box size="0.007 0.06 0.015" />
+        </geometry>
+      </collision>
+      <visual>
+        <origin xyz="0 0 0" rpy="0 0 0" />
+        <geometry>
+          <box size="0.007 0.06 0.015"  />
+        </geometry>
+      </visual>
+      <inertial>
+        <mass value="0.008" />
+        <origin xyz="0 0 0" rpy="0 0 0" />
+        <inertia ixx="1e-6" ixy="0" ixz="0" iyy="1e-6" iyz="0" izz="1e-6" />
+      </inertial>
+    </link>
+    <joint name="${namespace}_picoflexx_sensor_joint" type="fixed">
+      <xacro:insert_block name="origin" />
+      <parent link="${parent_link}" />
+      <child link="${namespace}/picoflexx_link" />
+    </joint>
+    <!-- Depth Sensor -->
+    <xacro:if value="${enable_depth}">
+      <xacro:picoflexx_depth_macro
+        namespace="${namespace}" parent_link="${namespace}/picoflexx_link"
+        camera_suffix="depth" frame_rate="10.0" max_range="4.0">
+        <origin xyz="0.015 0.055 0.0065" rpy="0 0 0" />
+      </xacro:picoflexx_depth_macro>
+    </xacro:if>
+    <xacro:if value="${enable_ground_truth}">
+      <!-- Odometry Sensor -->
+      <xacro:odometry_plugin_macro
+        namespace="${namespace}/ground_truth"
+        odometry_sensor_suffix=""
+        parent_link="${namespace}/picoflexx_link"
+        pose_topic="pose"
+        pose_with_covariance_topic="pose_with_covariance"
+        position_topic="position"
+        transform_topic="transform"
+        odometry_topic="odometry"
+        parent_frame_id="world"
+        child_frame_id="${namespace}/base_link"
+        mass_odometry_sensor="0.00001"
+        measurement_divisor="1"
+        measurement_delay="0"
+        unknown_delay="0.0"
+        noise_normal_position="0 0 0"
+        noise_normal_quaternion="0 0 0"
+        noise_normal_linear_velocity="0 0 0"
+        noise_normal_angular_velocity="0 0 0"
+        noise_uniform_position="0 0 0"
+        noise_uniform_quaternion="0 0 0"
+        noise_uniform_linear_velocity="0 0 0"
+        noise_uniform_angular_velocity="0 0 0"
+        enable_odometry_map="false"
+        odometry_map=""
+        image_scale="">
+        <inertia ixx="0.00001" ixy="0.0" ixz="0.0" iyy="0.00001" iyz="0.0" izz="0.00001" /> <!-- [kg m^2] [kg m^2] [kg m^2] [kg m^2] [kg m^2] [kg m^2] -->
+        <origin xyz="0.0 0.0 0.0" rpy="0.0 0.0 0.0" />
+      </xacro:odometry_plugin_macro>
+    </xacro:if>
+  </xacro:macro>
   <xacro:macro name="ground_truth_imu_and_odometry" params="namespace parent_link">
     <!-- Mount an IMU providing ground truth. -->

File: rotors_description/urdf/hummingbird_base.xacro (robot description, xacro)
@@ -39,3 +39,8 @@
       wait_to_record_bag="$(arg wait_to_record_bag)" />
   </xacro:if>
+  <!-- Add an 0S0-128 lidar -->
+  <xacro:include filename="$(find lidar_description)/urdf/OS0-128.urdf.xacro"/>
+  <xacro:OS0-128 parent="${namespace}/base_link" name="${namespace}/velodyne" topic="velodyne_points" hz="10" lasers="32" samples="440" collision_range="0.3" min_range="0.3" max_range="50.0">
+    <origin xyz="0 0 0.04" rpy="0 0 0" />
+  </xacro:OS0-128>
 </robot>

File: rotors_description/urdf/pelican_base.xacro (robot description, xacro)
@@ -20,4 +20,10 @@
   <!-- Instantiate pelican "mechanics" -->
   <xacro:include filename="$(find rotors_description)/urdf/pelican.xacro" />
+  <xacro:include filename="$(find realsense2_description)/urdf/_d435.urdf.xacro"/>
+  <xacro:include filename="$(find rotors_description)/urdf/rplidar.xacro"/>
+  <xacro:include filename="$(find rotors_description)/urdf/sbl.xacro" />
+  <xacro:sensor_rplidar parent="${namespace}/base_link" topics_ns="${namespace}/rplidar">
+    <origin xyz="0 0 0.2" rpy="0 0 0"/>
+  </xacro:sensor_rplidar>
   <!-- Instantiate a controller. -->
   <xacro:controller_plugin_macro namespace="${namespace}" imu_sub_topic="imu" />
