Commit message: sbl addition

File: rotors_description/urdf/hummingbird_base.xacro (robot description, xacro)
@@ -20,4 +20,5 @@
   <!-- Instantiate hummingbird "mechanics" -->
   <xacro:include filename="$(find rotors_description)/urdf/hummingbird.xacro" />
+  <xacro:include filename="$(find rotors_description)/urdf/sbl.xacro" />
   <!-- Instantiate a controller. -->
   <xacro:controller_plugin_macro namespace="${namespace}" imu_sub_topic="imu" />

File: rotors_description/urdf/pelican_base.xacro (robot description, xacro)
@@ -20,5 +20,5 @@
   <!-- Instantiate pelican "mechanics" -->
   <xacro:include filename="$(find rotors_description)/urdf/pelican.xacro" />
-  <xacro:include filename="$(find realsense2_description)/urdf/_d435.urdf.xacro"/>
+  <!-- <xacro:include filename="$(find realsense2_description)/urdf/_d435.urdf.xacro"/> -->
   <xacro:include filename="$(find rotors_description)/urdf/rplidar.xacro"/>
   <xacro:include filename="$(find rotors_description)/urdf/sbl.xacro" />

File: rotors_description/urdf/sbl.xacro (robot description, xacro)
@@ -17,5 +17,6 @@
 </link>
 <joint name="sbl_joint" type="fixed">
-    <parent link="pelican/base_link"/>
+    <!-- <parent link="pelican/base_link"/> -->
+    <parent link="hummingbird/base_link"/>
     <child link="sbl"/>
     <origin xyz="0.0 0.0 -0.1" rpy="0 1.57 0"/>
@@ -50,5 +51,5 @@
         </ray>
         <plugin filename="libgazebo_ros_range.so" name="gazebo_ros_range">
-            <topicName>sbl_down_range</topicName>
+            <topicName>sbl</topicName>
             <frameName>sbl</frameName>
             <gaussianNoise>0.000</gaussianNoise>
